File: smd-smores-pcb.kicad_sch (KiCad schematic)
At the start: 0 parts

Commit message: Basic schematic design without peripherals
Parts:
- added C1, C11, C15, C2, C20, C21: 4.7u, Capacitor_SMD:C_0402_1005Metric, symbol Device:C
- added C10: 820p, Capacitor_SMD:C_0402_1005Metric, symbol Device:C
- added C12, C13: 1p, Capacitor_SMD:C_0402_1005Metric, symbol Device:C
- added C14: 1.5p, Capacitor_SMD:C_0402_1005Metric, symbol Device:C
- added C16, C17, C18, C24, C25, C8: 100n, Capacitor_SMD:C_0402_1005Metric, symbol Device:C
- added C19, C23, C3: 1u, Capacitor_SMD:C_0402_1005Metric, symbol Device:C
- added C22: 47n, Capacitor_SMD:C_0402_1005Metric, symbol Device:C
- added C26: 2.2u, Capacitor_SMD:C_0402_1005Metric, symbol Device:C
- added C4, C5, C6, C7: 12p, Capacitor_SMD:C_0402_1005Metric, symbol Device:C
- added C9: 100p, Capacitor_SMD:C_0402_1005Metric, symbol Device:C
- added D1: LED_ORANGE, symbol Device:LED
- added L1: 3.9n, symbol Device:L
- added L2, L3: 10u, symbol Device:L
- added L4: 15n, symbol Device:L
- added R1, R2, R3, R5, R6: 10k, Resistor_SMD:R_0402_1005Metric, symbol Device:R
- added R10, R7, R8, R9: 4.7k, Resistor_SMD:R_0402_1005Metric, symbol Device:R
- added R4: 0, Resistor_SMD:R_1206_3216Metric, symbol Device:R
- added U1: nRF52840, Package_DFN_QFN:Nordic_AQFN-73-1EP_7x7mm_P0.5mm, symbol MCU_Nordic:nRF52840
- added U2: BQ24075RGT, Package_DFN_QFN:VQFN-16-1EP_3x3mm_P0.5mm_EP1.6x1.6mm, symbol Battery_Management:BQ24075RGT
- added U3: ICM-45686, ICM-45686:IC_ICM-45686, symbol ICM-45686:ICM-45686
- added U4: QMC6309, QMC6309:IC_QMC6309, symbol QMC6309:QMC6309
- added Y1: 32MHz, symbol Device:Crystal_GND2
- added Y2: 32.768kHz, symbol Device:Crystal
- added Y3: SG-8018CE, Oscillator:Oscillator_SMD_SeikoEpson_SG8002CE-4Pin_3.2x2.5mm, symbol Oscillator:SG-8002CE
Connections:
- new net: C22.1, C23.1, L4.2, U1.B5 (DEC4), U1.E24 (DEC6)
- new net: C8.1, U1.C1 (DEC1)
- new net: C11.1, U1.AC5 (DECUSB)
- new net: C9.1, U1.D23 (DEC3)
- new net: C7.2, U1.F2 (XL2/P0.01), Y2.2
- new net: C5.2, U1.A23 (XC2), Y1.3
- new net: L2.1, U1.AB2 (DCCH)
- new net: C4.2, U1.B24 (XC1), Y1.1
- new net: L3.1, U1.B3 (DCC)
- new net: C6.2, U1.D2 (XL1/P0.00), Y2.1
- new net: C12.1, L1.2, U1.H23 (ANT)
- new net: C10.1, U1.N24 (DEC5)
- new net: D1.1 (K), U2.9 (~{CHG})
- new net: D1.2 (A), R3.1
- new net: R2.1, U2.1 (TS)
- new net: L3.2, L4.1
- new net: C13.1, L1.1, R4.2
- new net: R1.2, U2.16 (ISET)
- new net 3V3: C24.1, C25.1, C26.1, R10.1, R5.1, R6.1, R7.1, R8.1, R9.1, U1.AD12 (P0.17), U3.5 (VDDIO), U3.8 (VDD), U4.B1 (VDD), Y3.4 (Vcc)
- new net ANTENNA: C14.1, R4.1
- new net BLED: U1.AD10 (P0.15)
- new net CLK: U3.9 (INT2), Y3.3 (OUT)
- new net CLKCTL: U1.B19 (P1.11), Y3.1 (OE)
- new net CS: R9.2, U1.AD22 (TRACEDATA0/P1.00), U3.12 (CSB)
- new net GND: C1.2, C10.2, C11.2, C13.2, C14.2, C15.2, C16.2, C17.2, C18.2, C19.2, C2.2, C20.2, C21.2, C22.2, C23.2, C24.2, C25.2, C26.2, C3.2, C4.1, C5.1, C6.1, C7.1, C8.2, C9.2, R1.1, R2.2, U1.B7 (VSS), U1.EP (VSS), U2.15 (SYSOFF), U2.17 (VSS), U2.4 (~{CE}), U2.5 (EN2), U2.8 (VSS), U3.6 (GND), U4.A1 (VSS), Y1.2, Y3.2 (GND)
- new net INT1: U1.A12 (AIN0/P0.02), U3.4 (INT1)
- new net RESET: U1.AC11 (P0.16), U1.AC13 (P0.18/~{RESET}), U1.AC9 (P0.14)
- new net SCL: R7.2, U1.AD18 (P0.22), U3.13 (SCX)
- new net SCX: R5.2, U3.3 (ASCX), U4.A2 (SCL)
- new net SDA: R8.2, U1.AD20 (P0.24), U3.14 (SDX)
- new net SDO: R10.2, U1.T2 (TRACEDATA2/P0.11), U3.1 (SDO)
- new net SDX: R6.2, U3.2 (ASDX), U4.B2 (SDA)
- new net SW0: U1.L1 (P0.06)
- new net SWC: U1.AA24 (SWDCLK)
- new net SWD: U1.AC24 (SWDIO)
- new net VBAT: C1.1, U2.2 (BAT), U2.3 (BAT)
- new net VBUS: C21.1, C3.1, U1.AD2 (VBUS), U2.13 (IN)
- new net VDDH: C2.1, C20.1, R3.2, U1.Y2 (VDDH), U2.10 (OUT), U2.11 (OUT), U2.6 (EN1)
- new net VDD_NRF: C15.1, C16.1, C17.1, C18.1, C19.1, L2.2, U1.A22 (VDD), U1.AD14 (VDD), U1.AD23 (VDD), U1.B1 (VDD), U1.W1 (VDD)
- new net VSS_PA: C12.2, U1.F23 (VSS_PA)
- no-connect marks 0 -> 43
Other:
- note added: "BQ24075RGT Charging IC"
- note added: "ICM-45686 based on KOUNOLAB's Module"
- note added: "nRF52840-QIAA-R Pin Configuration"

Commit message: Mid design v1
Parts:
- added D2: LED_BLUE, LED_SMD:LED_0402_1005Metric, symbol Device:LED
- added R11: 1k, Resistor_SMD:R_0402_1005Metric, symbol Device:R
- D1: footprint (none) -> LED_SMD:LED_0402_1005Metric
- L1, L4: footprint (none) -> Inductor_SMD:L_0402_1005Metric
- L2, L3: footprint (none) -> Inductor_SMD:L_0603_1608Metric
- Y1: footprint (none) -> Crystal:Crystal_SMD_3225-4Pin_3.2x2.5mm
- Y2: footprint (none) -> Crystal:Crystal_SMD_3215-2Pin_3.2x1.5mm
Connections:
- net GND: now also R11.2
- net RESET: no longer U1.AC13 (P0.18/~{RESET})
- net BLED: no longer names the net of U1.AD10 (P0.15)
- net BLED: now also D2.2 (A)
- new net: D2.1 (K), R11.1
Changed lines of the file:
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@@
 	(wire
 		(pts
+			(xy 125.73 105.41) (xy 139.7 105.41)
+		)
+		(stroke
+			(width 0)
+			(type default)
+		)
+	)
+	(wire
+		(pts
 			(xy 137.16 73.66) (xy 144.78 73.66)
 		)
@@
 		)
 	)
-	(global_label "BLED"
-		(shape input)
-		(at 125.73 105.41 0)
-		(fields_autoplaced yes)
-		(effects
-			(font
-				(size 1.27 1.27)
-				(thickness 0.1588)
-			)
-			(justify left)
-		)
-		(property "Intersheetrefs" "${INTERSHEET_REFS}"
-			(at 133.4323 105.41 0)
-			(effects
-				(font
-					(size 1.27 1.27)
-				)
-				(justify left)
-				(hide yes)
-			)
-		)
-	)
 	(global_label "SDX"
 		(shape input)
@@
 		)
 	)
-	(global_label "RESET"
-		(shape input)
-		(at 59.69 173.99 180)
-		(fields_autoplaced yes)
-		(effects
-			(font
-				(size 1.27 1.27)
-			)
-			(justify right)
-		)
-		(property "Intersheetrefs" "${INTERSHEET_REFS}"
-			(at 50.9597 173.99 0)
-			(effects
-				(font
-					(size 1.27 1.27)
-				)
-				(justify right)
-				(hide yes)
-			)
-		)
-	)
 	(global_label "CS"
 		(shape input)
@@
 		)
 	)
-	(global_label "VDD_NRF"
-		(shape input)
-		(at 92.71 59.69 90)
-		(fields_autoplaced yes)
-		(effects
-			(font
-				(size 1.27 1.27)
-			)
-			(justify left)
-		)
-		(property "Intersheetrefs" "${INTERSHEET_REFS}"
-			(at 92.71 48.4195 90)
-			(effects
-				(font
-					(size 1.27 1.27)
-				)
-				(justify left)
-				(hide yes)
-			)
-		)
-	)
 	(global_label "3V3"
 		(shape input)
@@
 		)
 	)
+	(global_label "VDD_NRF"
+		(shape input)
+		(at 92.71 59.69 90)
+		(fields_autoplaced yes)
+		(effects
+			(font
+				(size 1.27 1.27)
+			)
+			(justify left)
+		)
+		(property "Intersheetrefs" "${INTERSHEET_REFS}"
+			(at 92.71 48.4195 90)
+			(effects
+				(font
+					(size 1.27 1.27)
+				)
+				(justify left)
+				(hide yes)
+			)
+		)
+	)
 	(global_label "CS"
 		(shape input)
@@
 	)
 	(symbol
+		(lib_id "power:GND")
+		(at 139.7 120.65 0)
+		(mirror y)
+		(unit 1)
+		(exclude_from_sim no)
+		(in_bom yes)
+		(on_board yes)
+		(dnp no)
+		(fields_autoplaced yes)
+		(property "Reference" "#PWR030"
+			(at 139.7 127 0)
+			(effects
+				(font
+					(size 1.27 1.27)
+				)
+				(hide yes)
+			)
+		)
+		(property "Value" "GND"
+			(at 139.7 125.73 0)
+			(effects
+				(font
+					(size 1.27 1.27)
+				)
+			)
+		)
+		(property "Footprint" ""
+			(at 139.7 120.65 0)
+			(effects
+				(font
+					(size 1.27 1.27)
+				)
+				(hide yes)
+			)
+		)
+		(property "Datasheet" ""
+			(at 139.7 120.65 0)
+			(effects
+				(font
+					(size 1.27 1.27)
+				)
+				(hide yes)
+			)
+		)
+		(property "Description" "Power symbol creates a global label with name \"GND\" , ground"
+			(at 139.7 120.65 0)
+			(effects
+				(font
+					(size 1.27 1.27)
+				)
+				(hide yes)
+			)
+		)
+		(pin "1"
+		)
+		(instances
+			(project "smd-smores-pcb"
+				(path "/496e661b-dfd3-4b8a-a125-26ec39d316c4"
+					(reference "#PWR030")
+					(unit 1)
+				)
+			)
+		)
+	)
+	(symbol
 		(lib_id "Device:C")
 		(at 139.7 262.89 0)
@@
 			)
 		)
-		(property "Footprint" ""
+		(property "Footprint" "LED_SMD:LED_0402_1005Metric"
 			(at 99.06 261.62 0)
 			(effects
@@
 			)
 		)
-		(property "Footprint" ""
+		(property "Footprint" "Inductor_SMD:L_0402_1005Metric"
 			(at 114.3 53.34 0)
 			(effects
@@
 			)
 		)
-		(property "Footprint" ""
+		(property "Footprint" "Inductor_SMD:L_0603_1608Metric"
 			(at 109.22 59.69 0)
 			(effects
@@
 			)
 		)
-		(property "Footprint" ""
+		(property "Footprint" "Crystal:Crystal_SMD_3225-4Pin_3.2x2.5mm"
 			(at 53.34 130.81 0)
 			(effects
@@
 			)
 		)
-		(property "Footprint" ""
+		(property "Footprint" "Inductor_SMD:L_0402_1005Metric"
 			(at 54.61 85.09 0)
 			(effects
@@
 			)
 		)
-		(property "Footprint" ""
+		(property "Footprint" "Inductor_SMD:L_0603_1608Metric"
 			(at 106.68 53.34 0)
 			(effects
@@
 	)
 	(symbol
+		(lib_id "Device:LED")
+		(at 139.7 109.22 90)
+		(unit 1)
+		(exclude_from_sim no)
+		(in_bom yes)
+		(on_board yes)
+		(dnp no)
+		(property "Reference" "D2"
+			(at 146.05 108.966 0)
+			(effects
+				(font
+					(size 1.27 1.27)
+				)
+			)
+		)
+		(property "Value" "LED_BLUE"
+			(at 143.51 109.22 0)
+			(effects
+				(font
+					(size 1.27 1.27)
+				)
+			)
+		)
+		(property "Footprint" "LED_SMD:LED_0402_1005Metric"
+			(at 139.7 109.22 0)
+			(effects
+				(font
+					(size 1.27 1.27)
+				)
+				(hide yes)
+			)
+		)
+		(property "Datasheet" "~"
+			(at 139.7 109.22 0)
+			(effects
+				(font
+					(size 1.27 1.27)
+				)
+				(hide yes)
+			)
+		)
+		(property "Description" "Light emitting diode"
+			(at 139.7 109.22 0)
+			(effects
+				(font
+					(size 1.27 1.27)
+				)
+				(hide yes)
+			)
+		)
+		(property "Sim.Pins" "1=K 2=A"
+			(at 139.7 109.22 0)
+			(effects
+				(font
+					(size 1.27 1.27)
+				)
+				(hide yes)
+			)
+		)
+		(pin "2"
+		)
+		(pin "1"
+		)
+		(instances
+			(project "smd-smores-pcb"
+				(path "/496e661b-dfd3-4b8a-a125-26ec39d316c4"
+					(reference "D2")
+					(unit 1)
+				)
+			)
+		)
+	)
+	(symbol
 		(lib_id "Device:Crystal")
 		(at 137.16 68.58 270)
@@
 			)
 		)
-		(property "Footprint" ""
+		(property "Footprint" "Crystal:Crystal_SMD_3215-2Pin_3.2x1.5mm"
 			(at 137.16 68.58 0)
 			(effects
@@
 					(unit 1)
 				)
+			)
+		)
+	)
+	(symbol
+		(lib_id "Device:R")
+		(at 139.7 116.84 0)
+		(unit 1)
+		(exclude_from_sim no)
+		(in_bom yes)
+		(on_board yes)
+		(dnp no)
+		(fields_autoplaced yes)
+		(property "Reference" "R11"
+			(at 142.24 115.5699 0)
+			(effects
+				(font
+					(size 1.27 1.27)
+				)
+				(justify left)
+			)
+		)
+		(property "Value" "1k"
+			(at 142.24 118.1099 0)
+			(effects
+				(font
+					(size 1.27 1.27)
+				)
+				(justify left)
+			)
+		)
+		(property "Footprint" "Resistor_SMD:R_0402_1005Metric"
+			(at 137.922 116.84 90)
+			(effects
+				(font
+					(size 1.27 1.27)
+				)
+				(hide yes)
+			)
+		)
+		(property "Datasheet" "~"
+			(at 139.7 116.84 0)
+			(effects
+				(font
+					(size 1.27 1.27)
+				)
+				(hide yes)
+			)
+		)
+		(property "Description" "Resistor"
+			(at 139.7 116.84 0)
+			(effects
+				(font
+					(size 1.27 1.27)
+				)
+				(hide yes)
+			)
+		)
+		(pin "1"
+		)
+		(pin "2"
+		)
+		(instances
+			(project "smd-smores-pcb"
+				(path "/496e661b-dfd3-4b8a-a125-26ec39d316c4"
+					(reference "R11")
+					(unit 1)
+				)
